File: zenga_pcb/lascheda.kicad_pcb (KiCad board)
At the start: 2 copper layers, 165.9 x 162.1 mm, 50 parts

Commit message: Finish first routing draft
Parts:
- added REF**: Jack_3.5mm_CUI_SJ1-3535NG_Horizontal, Connector_Audio:Jack_3.5mm_CUI_SJ1-3535NG_Horizontal, F.Cu at (212.8, 138.2)
- moved OLED1 10.2 mm to (192.1, 131.8)
- moved D24 7.21 mm to (209.1, 179.5), turned to 124.5 degrees
- moved D23 6.91 mm to (193.1, 163.2), turned to 133.5 degrees
- moved D22 6.80 mm to (175.0, 149.2), turned to 142.5 degrees
- moved S22 0.29 mm to (171.9, 153.2), turned to 142.5 degrees
- moved S23 0.27 mm to (189.5, 166.7), turned to 133.5 degrees
- moved S24 0.19 mm to (205.0, 182.4), turned to 124.5 degrees
Routing:
- net GP10: track 239.8 -> 300.5 mm, vias 4 -> 5
- net GP11: track 243.4 -> 290.1 mm
- net P3V3: track 0.00 -> 41.9 mm, vias 0 -> 1
- net GP0: track 0.00 -> 41.8 mm
- net GP1: track 0.00 -> 38.8 mm, vias 0 -> 1
- net GP13: track 169.1 -> 198.0 mm, vias 3 -> 4
- net GP12: track 311.4 -> 327.4 mm, vias 4 -> 5
- net GP28: track 173.1 -> 184.5 mm
- net GP26: track 115.1 -> 125.4 mm
- net GP15: track 116.3 -> 126.1 mm
- net GP27: track 145.9 -> 155.1 mm
- net GP29: track 190.2 -> 196.9 mm
- net indexouter_home: track 27.4 -> 32.9 mm
- net GP14: track 170.1 -> 164.6 mm
- net GP9: track 364.0 -> 360.6 mm
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- added copper zone on B.Cu, net GND
- added copper zone on F.Cu, net GND
